Commit message: Advances in urdf course

File: urdf_for_robot_modelling_ws/src/my_gurdy_description/urdf/gurdy_controllers.urdf (robot description, URDF)
Before this commit: robot gurdy, 11 links, 10 joints
Joints:
- joint head_upperlegM1_joint: limit lower=-1.5 upper=1.5 effort=1 velocity=0.005 -> lower=-1.55 upper=0 effort=1 velocity=0.005
- joint head_upperlegM2_joint: limit lower=-1.5 upper=1.5 effort=1 velocity=0.005 -> lower=-1.55 upper=0 effort=1 velocity=0.005
- joint head_upperlegM3_joint: limit lower=-1.5 upper=1.5 effort=1 velocity=0.005 -> lower=-1.55 upper=0 effort=1 velocity=0.005
- joint upperlegM1_lowerlegM1_joint: limit lower=-1.6 upper=1.6 effort=1 velocity=0.005 -> lower=-2.9 upper=1.57 effort=1 velocity=0.005
- joint upperlegM2_lowerlegM2_joint: limit lower=-1.6 upper=1.6 effort=1 velocity=0.005 -> lower=-2.9 upper=1.57 effort=1 velocity=0.005
- joint upperlegM3_lowerlegM3_joint: limit lower=-1.6 upper=1.6 effort=1 velocity=0.005 -> lower=-2.9 upper=1.57 effort=1 velocity=0.005
