Commit message: Change z-joint for upperleg to rotate around the joint, not the centre

File: urdf_for_robot_modelling_ws/src/my_gurdy_description/urdf/gurdy_extra_joint.urdf (robot description, URDF)
Before this commit: robot gurdy, 12 links, 11 joints
Links:
- added link virtual_M2_link
- added link virtual_M3_link
Joints:
- added joint Z_M2_joint: type revolute, parent virtual_M2_link, child upperleg_M2_link, origin xyz=0 0 0 rpy=0 0 0, axis 0 0 1, limit lower=-0.7854 upper=0.7854 effort=1 velocity=0.005
- added joint Z_M3_joint: type revolute, parent virtual_M3_link, child upperleg_M3_link, origin xyz=0 0 0 rpy=0 0 0, axis 0 0 1, limit lower=-0.7854 upper=0.7854 effort=1 velocity=0.005
- joint Z_M1_joint: child virtual_M1_link -> upperleg_M1_link; limit lower=-3.141592 upper=3.141592 effort=1 velocity=0.005 -> lower=-0.7854 upper=0.7854 effort=1 velocity=0.005; parent head_link -> virtual_M1_link
- joint head_upperlegM1_joint: child upperleg_M1_link -> virtual_M1_link; parent virtual_M1_link -> head_link
- joint head_upperlegM2_joint: child upperleg_M2_link -> virtual_M2_link

Commit message: Add inertia and mass to virtual links to appear in Gazebo. Change axis

File: urdf_for_robot_modelling_ws/src/my_gurdy_description/urdf/gurdy_extra_joint.urdf (robot description, URDF)
Before this commit: robot gurdy, 14 links, 13 joints
Links:
- link virtual_M1_link: mass None -> 0.001
- link virtual_M2_link: mass None -> 0.001
- link virtual_M3_link: mass None -> 0.001
Joints:
- joint Z_M1_joint: axis 0 0 1 -> 1 0 0
- joint Z_M2_joint: axis 0 0 1 -> 1 0 0
- joint Z_M3_joint: axis 0 0 1 -> 1 0 0
- joint head_upperlegM3_joint: child upperleg_M3_link -> virtual_M3_link

Commit message: Correct rotation of z-joint

File: urdf_for_robot_modelling_ws/src/my_gurdy_description/urdf/gurdy_extra_joint.urdf (robot description, URDF)
Before this commit: robot gurdy, 14 links, 13 joints
Joints:
- joint Z_M1_joint: axis 1 0 0 -> 0 0 1; child upperleg_M1_link -> virtual_M1_link; origin xyz=0 0 0 rpy=0 0 0 -> xyz=-0.02165 -0.0125 -0.008 rpy=3.14159 0 0.523599; parent virtual_M1_link -> head_link
- joint head_upperlegM1_joint: child virtual_M1_link -> upperleg_M1_link; origin xyz=-0.02165 -0.0125 -0.008 rpy=3.14159 0 0.523599 -> xyz=0 0 0 rpy=0 0 0; parent head_link -> virtual_M1_link

Commit message: Extend urdf joint changes to the 3 joints

File: urdf_for_robot_modelling_ws/src/my_gurdy_description/urdf/gurdy_extra_joint.urdf (robot description, URDF)
Before this commit: robot gurdy, 14 links, 13 joints
Joints:
- joint Z_M2_joint: axis 1 0 0 -> 0 0 1; child upperleg_M2_link -> virtual_M2_link; origin xyz=0 0 0 rpy=0 0 0 -> xyz=0.02165 -0.0125 -0.008 rpy=3.14159 0 2.61799; parent virtual_M2_link -> head_link
- joint Z_M3_joint: axis 1 0 0 -> 0 0 1; child upperleg_M3_link -> virtual_M3_link; origin xyz=0 0 0 rpy=0 0 0 -> xyz=0 0.025 -0.008 rpy=3.14159 0 -1.5708; parent virtual_M3_link -> head_link
- joint head_upperlegM2_joint: child virtual_M2_link -> upperleg_M2_link; origin xyz=0.02165 -0.0125 -0.008 rpy=3.14159 0 2.61799 -> xyz=0 0 0 rpy=0 0 0; parent head_link -> virtual_M2_link
- joint head_upperlegM3_joint: child virtual_M3_link -> upperleg_M3_link; origin xyz=0 0.025 -0.008 rpy=3.14159 0 -1.5708 -> xyz=0 0 0 rpy=0 0 0; parent head_link -> virtual_M3_link

Commit message: Create xacros

File: urdf_for_robot_modelling_ws/src/my_gurdy_description/urdf/gurdy_extra_joint.urdf (robot description, URDF)
Before this commit: robot gurdy, 14 links, 13 joints
Joints:
- removed joint Z_M1_joint
- removed joint Z_M2_joint
- removed joint Z_M3_joint
- added joint z_rotary_M1_joint: type revolute, parent head_link, child virtual_M1_link, origin xyz=-0.02165 -0.0125 -0.008 rpy=3.14159 0 0.523599, axis 0 0 1, limit lower=-0.7854 upper=0.7854 effort=1 velocity=0.005
- added joint z_rotary_M2_joint: type revolute, parent head_link, child virtual_M2_link, origin xyz=0.02165 -0.0125 -0.008 rpy=3.14159 0 2.61799, axis 0 0 1, limit lower=-0.7854 upper=0.7854 effort=1 velocity=0.005
- added joint z_rotary_M3_joint: type revolute, parent head_link, child virtual_M3_link, origin xyz=0 0.025 -0.008 rpy=3.14159 0 -1.5708, axis 0 0 1, limit lower=-0.7854 upper=0.7854 effort=1 velocity=0.005
