Commit message: Correct xacro issues

File: urdf_for_robot_modelling_ws/src/my_gurdy_description/robots/gurdy.urdf.xacro (robot description, xacro)
@@ -6,4 +6,17 @@
         </plugin>
     </gazebo>
+    <!-- * * * XACROS * * * -->
+    <xacro:property name="rotary_joint_lower_limit" value="-0.9" />
+    <xacro:property name="rotary_joint_upper_limit" value="0.9" />
+    <xacro:property name="rotary_joint_effort_limit" value="1" />
+    <xacro:property name="rotary_joint_velocity_limit" value="0.005" />
+    <xacro:property name="upperleg_joint_lower_limit" value="-2.9" />
+    <xacro:property name="upperleg_joint_upper_limit" value="1.57" />
+    <xacro:property name="upperleg_joint_effort_limit" value="1" />
+    <xacro:property name="upperleg_joint_velocity_limit" value="0.005" />
+    <xacro:property name="lowerleg_joint_lower_limit" value="-1.55" />
+    <xacro:property name="lowerleg_joint_upper_limit" value="0" />
+    <xacro:property name="lowerleg_joint_effort_limit" value="1" />
+    <xacro:property name="lowerleg_joint_velocity_limit" value="0.005" />
     <!-- * * * MACROS * * * -->
     <!-- Rotary Joints -->
@@ -16,5 +29,5 @@
             </inertial>
         </link>
-    </xacro>
+    </xacro:macro>
     <xacro:macro name="z_rotary_transmission" params="number">
         <transmission name="tran${number}">
@@ -28,5 +41,5 @@
             </actuator>
         </transmission>
-    </xacro>
+    </xacro:macro>
     <!-- Upperlegs -->
     <xacro:macro name="upperleg_link" params="number">
@@ -50,5 +63,5 @@
             </visual>
         </link>
-    </xacro>
+    </xacro:macro>
     <xacro:macro name="upperleg_joint" params="number">
         <joint name="head_upperlegM${number}_joint" type="revolute">
@@ -66,5 +79,5 @@
             <axis xyz="0 1 0"/> <!-- The axis of rotation are with reference to the axis of the joint, not the global reference frame. Hence, these are the global reference axes after the rpy transformation - You can visualize them in RViz -->
         </joint>
-    </xacro>
+    </xacro:macro>
     <xacro:macro name="upperleg_transmission" params="number">
         <transmission name="tran${number}">
@@ -78,5 +91,5 @@
             </actuator>
         </transmission>
-    </xacro>
+    </xacro:macro>
     <!-- Lowerlegs -->
     <xacro:macro name="lowerleg_link" params="number">
@@ -100,5 +113,5 @@
             </visual>
         </link>
-    </xacro>
+    </xacro:macro>
     <xacro:macro name="lowerleg_joint" params="number">
         <joint name="upperlegM${number}_lowerlegM${number}_joint" type="revolute">
@@ -116,5 +129,5 @@
             <axis xyz="0 1 0"/>
         </joint>
-    </xacro>
+    </xacro:macro>
     <xacro:macro name="lowerleg_transmission" params="number">
         <transmission name="tran${number}">
@@ -128,5 +141,5 @@
             </actuator>
         </transmission>
-    </xacro>
+    </xacro:macro>
     <!-- Feet -->
     <xacro:macro name="foot_link" params="number">
@@ -150,5 +163,5 @@
             </visual>
         </link>
-    </xacro>
+    </xacro:macro>
     <xacro:macro name="foot_gazebo" params="number color">
         <gazebo reference="footM${number}_link">
@@ -159,5 +172,5 @@
             <material>Gazebo/${color}</material> <!-- This is the colour for the Gazebo simulation. Not applicable for dae files since the colours are embedded in the 3Dfile -->
         </gazebo>
-    </xacro>
+    </xacro:macro>
     <xacro:macro name="foot_joint" params="number">
         <joint name="lowerlegM${number}_footM${number}_joint" type="fixed">
@@ -166,18 +179,5 @@
             <origin xyz="0 0 0.06" rpy="0 0 0"/>
         </joint>
-    </xacro>
-    <!-- * * * XACROS * * * -->
-    <xacro:property name="rotary_joint_lower_limit" value="-0.9" />
-    <xacro:property name="rotary_joint_upper_limit" value="0.9" />
-    <xacro:property name="rotary_joint_effort_limit" value="1" />
-    <xacro:property name="rotary_joint_velocity_limit" value="0.005" />
-    <xacro:property name="upperleg_joint_lower_limit" value="-2.9" />
-    <xacro:property name="upperleg_joint_upper_limit" value="1.57" />
-    <xacro:property name="upperleg_joint_effort_limit" value="1" />
-    <xacro:property name="upperleg_joint_velocity_limit" value="0.005" />
-    <xacro:property name="lowerleg_joint_lower_limit" value="-1.55" />
-    <xacro:property name="lowerleg_joint_upper_limit" value="0" />
-    <xacro:property name="lowerleg_joint_effort_limit" value="1" />
-    <xacro:property name="lowerleg_joint_velocity_limit" value="0.005" />
+    </xacro:macro>
 	<!-- * * * LINK & JOINT DEFINITIONS * * * -->
     <!-- Base & Head -->
@@ -281,11 +281,11 @@
     <xacro:foot_link number="1"/>
     <xacro:foot_gazebo number="1" color="Red"/>
-    <xacro:foot_transmission number="1"/>
+    <xacro:foot_joint number="1"/>
     <xacro:foot_link number="2"/>
     <xacro:foot_gazebo number="2" color="Green"/>
-    <xacro:foot_transmission number="2"/>
+    <xacro:foot_joint number="2"/>
     <xacro:foot_link number="3"/>
     <xacro:foot_gazebo number="3" color="Blue"/>
-    <xacro:foot_transmission number="3"/>
+    <xacro:foot_joint number="3"/>
     <!-- * * * SENSORS * * * -->
     <!-- IMU -->
